Commit message: fix: change pkg name in urdf

File: urdf/roar.urdf (robot description, URDF)
Before this commit: robot roar, 11 links, 10 joints
Links:
- link base_link: geometry collision mesh filename=package://roar_simulation/meshes/base_link.STL; visual mesh filename=package://roar_simulation/meshes/base_link.STL
- link bogie_lhs: geometry collision mesh filename=package://roar_simulation/meshes/bogie_lhs.STL; visual mesh filename=package://roar_simulation/meshes/bogie_lhs.STL
- link bogie_rhs: geometry collision mesh filename=package://roar_simulation/meshes/bogie_rhs.STL; visual mesh filename=package://roar_simulation/meshes/bogie_rhs.STL
- link rocker_lhs: geometry collision mesh filename=package://roar_simulation/meshes/rocker_lhs.STL; visual mesh filename=package://roar_simulation/meshes/rocker_lhs.STL
- link rocker_rhs: geometry collision mesh filename=package://roar_simulation/meshes/rocker_rhs.STL; visual mesh filename=package://roar_simulation/meshes/rocker_rhs.STL
- link wheel_lhs_front: geometry collision mesh filename=package://roar_simulation/meshes/wheel_lhs_front.STL; visual mesh filename=package://roar_simulation/meshes/wheel_lhs_front.STL
- link wheel_lhs_mid: geometry collision mesh filename=package://roar_simulation/meshes/wheel_lhs_mid.STL; visual mesh filename=package://roar_simulation/meshes/wheel_lhs_mid.STL
- link wheel_lhs_rear: geometry collision mesh filename=package://roar_simulation/meshes/wheel_lhs_rear.STL; visual mesh filename=package://roar_simulation/meshes/wheel_lhs_rear.STL
- link wheel_rhs_front: geometry collision mesh filename=package://roar_simulation/meshes/wheel_rhs_front.STL; visual mesh filename=package://roar_simulation/meshes/wheel_rhs_front.STL
- link wheel_rhs_mid: geometry collision mesh filename=package://roar_simulation/meshes/wheel_rhs_mid.STL; visual mesh filename=package://roar_simulation/meshes/wheel_rhs_mid.STL
- link wheel_rhs_rear: geometry collision mesh filename=package://roar_simulation/meshes/wheel_rhs_rear.STL; visual mesh filename=package://roar_simulation/meshes/wheel_rhs_rear.STL

Commit message: fear: added camera to roar.urdf

File: urdf/roar.urdf (robot description, URDF)
Before this commit: robot roar_simulation, 11 links, 10 joints
Links:
- added link camera_link
- added link camera_optical_frame
Joints:
- added joint camera_joint: type fixed, parent base_link, child camera_link, origin xyz=0 0.3 0.35 rpy=0 0 1.570796
- added joint camera_optical_frame_joint: type fixed, parent camera_link, child camera_optical_frame, origin xyz=0 0 0 rpy=-1.570796 0 -1.570796

Commit message: feat: add zed  zed camera

File: urdf/roar.urdf (robot description, URDF)
Before this commit: robot roar_simulation, 13 links, 12 joints
Joints:
- joint camera_optical_frame_joint: origin xyz=0 0 0 rpy=-1.570796 0 -1.570796 -> xyz=0 0 0 rpy=-1.570796 0 0

Commit message: feat: updated the urdf file for the camera rotation

File: urdf/roar.urdf (robot description, URDF)
Before this commit: robot roar_simulation, 13 links, 12 joints
Links:
- removed link camera_optical_frame
- added link camera_depth_optical_frame, mass 0.001
- added link dummy_root
- link camera_link: mass None -> 0.001
Joints:
- removed joint camera_optical_frame_joint
- added joint camera_depth_optical_joint: type fixed, parent camera_link, child camera_depth_optical_frame, origin xyz=0 0 0 rpy=-1.57079632679 0 -1.57079632679
- added joint dummy_joint: type fixed, parent dummy_root, child base_link, origin xyz=0 0 0 rpy=0 0 0
- joint camera_joint: origin xyz=0 0.3 0.35 rpy=0 0 1.570796 -> xyz=0 0.3 0.35 rpy=0 0 1.57079632679
