Commit message: Repositioned switch, updated colors, and cleaned up workspace tracking

File: src/erc_panel_sim/urdf/panel.urdf.xacro (robot description, xacro)
@@ -1,7 +1,7 @@
 <?xml version="1.0"?>
 <robot name="erc_panel" xmlns:xacro="http://www.ros.org/wiki/xacro">
-<!-- <material name="silver">
-  <color rgba="0.700 0.700 0.700 1.000"/>
-</material> silver material defined here-->
+ <material name="dark_grey">
+  <color rgba="0.200 0.200 0.200 1.000"/>
+</material> <!-- dark grey material defined here for switches -->
   <!-- include switch macro -->
   <xacro:include filename="$(find switch_description)/urdf/rotary_control.xacro"/>
@@ -34,3 +34,7 @@
   <xacro:rotary_switch name="rotary_5" parent="panel_face"
     x="0.13" y="-0.007" z="-0.015"/>
+<!-- 2 large rotary switches -->
+<xacro:include filename="$(find rotary_description)/urdf/rotary.xacro"/>
+<xacro:rotary name="large_rotary_1" parent="panel_face" x="0.04" y="0.05" z="-0.15"/>
+<xacro:rotary name="large_rotary_2" parent="panel_face" x="0.125" y="0.05" z="-0.15"/>
 </robot>

File: src/switch_description/urdf/rotary_control.xacro (robot description, xacro)
@@ -1,5 +1,5 @@
 <?xml version="1.0" ?>
 <robot name="switch" xmlns:xacro="http://www.ros.org/wiki/xacro">
-<xacro:include filename="$(find switch_description)/urdf/switch_materials.xacro" />
+<!-- <xacro:include filename="$(find switch_description)/urdf/switch_materials.xacro" />  color defined in main xacro now-->
 <xacro:include filename="$(find switch_description)/urdf/switch.ros2control" />
 <xacro:include filename="$(find switch_description)/urdf/switch.gazebo" />
