Commit message: Fix URDF hierarchy, kinematic tree, and launch namespaces

File: src/erc_panel_sim/urdf/panel.urdf.xacro (robot description, xacro)
@@ -3,4 +3,7 @@
  <material name="dark_grey">
   <color rgba="0.500 0.500 0.500 1.000"/>
+</material>
+<material name="green">
+  <color rgba="0.0 1.0 0.0 1.0"/>
 </material> <!-- dark grey material defined here for switches -->
   <!-- include switch macro -->
@@ -25,13 +28,13 @@
   <!-- x:left/right y:forward/backward z:down -->
   <xacro:rotary_switch name="rotary_1" parent="panel_face"
-    x="-0.13" y="0.00" z="-0.015"/>
+    x="-0.13" y="0.005" z="-0.015"/>
   <xacro:rotary_switch name="rotary_2" parent="panel_face"
-    x="-0.065" y="0.00" z="-0.015"/>
+    x="-0.065" y="0.005" z="-0.015"/>
   <xacro:rotary_switch name="rotary_3" parent="panel_face"
-    x="0.000" y="0.00" z="-0.015"/>
+    x="0.000" y="0.005" z="-0.015"/>
   <xacro:rotary_switch name="rotary_4" parent="panel_face"
-    x="0.065" y="0.00" z="-0.015"/>
+    x="0.065" y="0.005" z="-0.015"/>
   <xacro:rotary_switch name="rotary_5" parent="panel_face"
-    x="0.13" y="0.00" z="-0.015"/>
+    x="0.13" y="0.005" z="-0.015"/>
 <!-- 2 large rotary switches -->
 <!-- x:left/right y:forward/backward z:down -->
@@ -60,3 +63,38 @@
 <xacro:socket name="socket_1" parent="panel_face" x="-0.07 " y="0" z="-0.1"/>
 <xacro:socket name="socket_2" parent="panel_face" x="-0.07" y="0" z="-0.135"/>
+<!--indicators-->
+<xacro:include filename="$(find led_indicator_description)/urdf/led_indicator.xacro"/>
+<xacro:led_indicator name="indicator_1" parent="panel_face" x="-0.08" y="0.008" z="0.2"/>
+<xacro:led_indicator name="indicator_2" parent="panel_face" x="-0.04" y="0.008" z="0.2"/>
+<xacro:led_indicator name="indicator_3" parent="panel_face" x="0.0" y="0.008" z="0.2"/>
+<xacro:led_indicator name="indicator_4" parent="panel_face" x="0.04" y="0.008" z="0.2"/>
+<xacro:led_indicator name="indicator_5" parent="panel_face" x="0.08" y="0.008" z="0.2"/>
+<!-- main switch -->
+<!--x:right y:in z:up-->
+<xacro:include filename="$(find main_switch_description)/urdf/main_switch.xacro"/>
+<xacro:main_switch name="main_switch" parent="panel_face" x="0.12" y="0.01" z="0.095"/>
+<!--slab holder-->
+<xacro:include filename="$(find slab_description)/urdf/slab.xacro"/>
+<xacro:slab name="slab" parent="panel_face" x="0.055" y="0.075" z="-0.1888"/>
+<!-- aruco markers -->
+<xacro:include filename="$(find aruco_description)/urdf/aruco_marker.xacro" />
+<xacro:aruco_marker
+  name="aruco_top_left"
+  parent="panel_face"
+  x="-0.13" y="-0.001" z="0.19"
+  texture_file="marker_id_1.png" />
+<xacro:aruco_marker
+  name="aruco_top_right"
+  parent="panel_face"
+  x="0.13" y="-0.001" z="0.19"
+  texture_file="marker_id_2.png" />
+<xacro:aruco_marker
+  name="aruco_bottom_left"
+  parent="panel_face"
+  x="-0.13" y="-0.001" z="-0.19"
+  texture_file="marker_id_3.png" />
+<!-- electromagnet-->
+<xacro:include filename="$(find electromagnet_description)/urdf/electromagnet.xacro" />
+<xacro:electromagnet name="electromagnet" parent="panel_face"
+  x="-0.193" y="0.02" z="-0.015"/>
 </robot>

File: src/row_description/urdf/row.xacro (robot description, xacro)
@@ -29,5 +29,5 @@
     <origin xyz="-4.057487931493324e-07 0.0003920169114006583 -0.004603424306532057" rpy="0 0 0"/>
     <mass value="0.00434807010112859"/>
-    <inertia ixx="0.0" iyy="0.0" izz="0.0" ixy="0.0" iyz="0.0" ixz="0.0"/>
+    <inertia ixx="2e-06" iyy="2e-06" izz="1e-06" ixy="-0.0" iyz="0.0" ixz="-0.0"/> <!-- copied from switch-->
   </inertial>
   <visual>

Commit message: fix: gravity

File: src/erc_panel_sim/urdf/panel.urdf.xacro (robot description, xacro)
@@ -10,13 +10,14 @@
   <xacro:include filename="$(find switch_description)/urdf/rotary_control.xacro"/>
   <!-- world anchor -->
-  <link name="world"/>
+<!--  <link name="world"/>
+commented world link so it would fall down in gazebo -->
   <!-- panel base -->
    <xacro:include filename="$(find panel_body_description)/urdf/panel_body.xacro"/>
  <!-- attach panel base to world -->
-   <joint name="world_to_panel" type="fixed">
+<!--   <joint name="world_to_panel" type="fixed">
   <parent link="world"/>
   <child link="panel_base_link"/>
   <origin xyz="0 0.0 0" rpy="0 0 0"/>
-</joint>
+</joint> -->
 <link name="panel_face"/>
 <joint name="panel_to_face" type="fixed"> <!--Added this to attach switches directly to the tilted panel face-->
